File: Project Architecture.kicad_sch (KiCad schematic)
At the start: 0 parts

Commit message: First Draft of the Schematic
Other:
- sheet Section A - Title A renamed Section A - Connectors
- sheet Section B - Title B renamed Section B - Arduino Mega
- added sheet Section C - LCL Selector (Section C - Title C.kicad_sch)
Changed lines of the file:
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@@
 (kicad_sch
-	(version 20231120)
+	(version 20250114)
 	(generator "eeschema")
-	(generator_version "8.0")
+	(generator_version "9.0")
 	(paper "A3")
 	(title_block
@@
 		(company "${COMPANY}")
 	)
-	(polyline
-		(pts
-			(xy 185.42 87.63) (xy 185.42 99.06)
-		)
-		(stroke
-			(width 0)
-			(type default)
-		)
-	)
-	(polyline
-		(pts
-			(xy 233.68 125.73) (xy 233.68 134.62)
-		)
-		(stroke
-			(width 0)
-			(type default)
-		)
-	)
-	(polyline
-		(pts
-			(xy 185.42 85.09) (xy 185.42 73.66)
-		)
-		(stroke
-			(width 0)
-			(type default)
-		)
-	)
-	(polyline
-		(pts
-			(xy 233.68 114.3) (xy 233.68 123.19)
-		)
-		(stroke
-			(width 0)
-			(type default)
-		)
-	)
 	(arc
 		(start 185.42 85.09)
@@
 	)
 	(arc
+		(start 185.43 166.38)
+		(mid 186.3251 166.7549)
+		(end 186.7 167.65)
+		(stroke
+			(width 0)
+			(type default)
+		)
+		(fill
+			(type none)
+		)
+	)
+	(arc
 		(start 233.7 125.71)
 		(mid 234.0749 124.8149)
@@
 	)
 	(arc
+		(start 186.7 165.11)
+		(mid 186.3251 166.0051)
+		(end 185.43 166.38)
+		(stroke
+			(width 0)
+			(type default)
+		)
+		(fill
+			(type none)
+		)
+	)
+	(arc
 		(start 233.7 134.6)
 		(mid 232.9561 136.3961)
@@
 	)
 	(arc
+		(start 186.7 153.68)
+		(mid 187.4439 151.8839)
+		(end 189.24 151.14)
+		(stroke
+			(width 0)
+			(type default)
+		)
+		(fill
+			(type none)
+		)
+	)
+	(arc
+		(start 189.24 181.62)
+		(mid 187.4498 180.8702)
+		(end 186.7 179.08)
+		(stroke
+			(width 0)
+			(type default)
+		)
+		(fill
+			(type none)
+		)
+	)
+	(arc
 		(start 185.42 73.66)
 		(mid 186.1639 71.8639)
@@
 		)
 	)
-	(text_box "Description"
+	(text "Page 5"
+		(exclude_from_sim no)
+		(at 226.06 133.35 0)
+		(effects
+			(font
+				(size 2.54 2.54)
+				(bold yes)
+				(color 100 70 50 1)
+			)
+			(justify right bottom)
+			(href "#5")
+		)
+	)
+	(text "Page 4"
+		(exclude_from_sim no)
+		(at 226.06 95.25 0)
+		(effects
+			(font
+				(size 2.54 2.54)
+				(bold yes)
+				(color 20 60 40 1)
+			)
+			(justify right bottom)
+			(href "#4")
+		)
+	)
+	(text_box "LCL Selector"
+		(exclude_from_sim no)
+		(at 165.1 160.02 0)
+		(size 17.145 5.08)
+		(margins 1.4287 1.4287 1.4287 1.4287)
+		(stroke
+			(width -0.0001)
+			(type solid)
+		)
+		(fill
+			(type none)
+		)
+		(effects
+			(font
+				(size 1.905 1.905)
+				(thickness 0.381)
+				(bold yes)
+				(color 0 0 0 1)
+			)
+			(justify right top)
+		)
+	)
+	(text_box "Power Entry and Connectors"
 		(exclude_from_sim no)
 		(at 166.37 83.82 0)
 		(size 17.145 5.08)
+		(margins 1.4287 1.4287 1.4287 1.4287)
 		(stroke
 			(width -0.0001)
-			(type default)
+			(type solid)
 		)
 		(fill
@@
 		)
 	)
-	(text_box "Description"
+	(text_box "Arduino Mega 2560"
 		(exclude_from_sim no)
 		(at 234.95 121.92 0)
 		(size 26.015 5.1)
+		(margins 1.4287 1.4287 1.4287 1.4287)
 		(stroke
 			(width -0.0001)
-			(type default)
+			(type solid)
 		)
 		(fill
@@
 		(at 144.78 21.59 0)
 		(size 130.81 12.7)
+		(margins 5.9999 5.9999 5.9999 5.9999)
 		(stroke
 			(width -0.0001)
@@
 		)
 	)
-	(text "Page 5"
-		(exclude_from_sim no)
-		(at 226.06 133.35 0)
-		(effects
-			(font
-				(size 2.54 2.54)
-				(bold yes)
-				(color 100 70 50 1)
-			)
-			(justify right bottom)
-			(href "#5")
-		)
-	)
-	(text "Page 4"
-		(exclude_from_sim no)
-		(at 226.06 95.25 0)
-		(effects
-			(font
-				(size 2.54 2.54)
-				(bold yes)
-				(color 20 60 40 1)
-			)
-			(justify right bottom)
-			(href "#4")
+	(polyline
+		(pts
+			(xy 186.7 165.11) (xy 186.7 153.68)
+		)
+		(stroke
+			(width 0)
+			(type default)
+		)
+	)
+	(polyline
+		(pts
+			(xy 186.7 167.65) (xy 186.7 179.08)
+		)
+		(stroke
+			(width 0)
+			(type default)
+		)
+	)
+	(polyline
+		(pts
+			(xy 185.42 87.63) (xy 185.42 99.06)
+		)
+		(stroke
+			(width 0)
+			(type default)
+		)
+	)
+	(polyline
+		(pts
+			(xy 233.68 125.73) (xy 233.68 134.62)
+		)
+		(stroke
+			(width 0)
+			(type default)
+		)
+	)
+	(polyline
+		(pts
+			(xy 185.42 85.09) (xy 185.42 73.66)
+		)
+		(stroke
+			(width 0)
+			(type default)
+		)
+	)
+	(polyline
+		(pts
+			(xy 233.68 114.3) (xy 233.68 123.19)
+		)
+		(stroke
+			(width 0)
+			(type default)
+		)
+	)
+	(sheet
+		(at 190.5 152.4)
+		(size 38.1 22.86)
+		(exclude_from_sim no)
+		(in_bom yes)
+		(on_board yes)
+		(dnp no)
+		(fields_autoplaced yes)
+		(stroke
+			(width 0.1524)
+			(type solid)
+		)
+		(fill
+			(color 0 194 194 1.0000)
+		)
+		(property "Sheetname" "Section C - LCL Selector"
+			(at 190.5 151.3709 0)
+			(effects
+				(font
+					(size 1.905 1.905)
+					(thickness 0.381)
+					(bold yes)
+				)
+				(justify left bottom)
+			)
+		)
+		(property "Sheetfile" "Section C - Title C.kicad_sch"
+			(at 190.5 175.8446 0)
+			(effects
+				(font
+					(size 1.27 1.27)
+				)
+				(justify left top)
+			)
+		)
+		(instances
+			(project "VPDCU_EGSE"
+				(path "/f9e05184-c88b-4a88-ae9c-ab2bdb32be7c/c5103ceb-5325-4a84-a025-9638a412984e"
+					(page "6")
+				)
+			)
 		)
 	)
@@
 		(at 190.5 114.3)
 		(size 36.83 20.32)
+		(exclude_from_sim no)
+		(in_bom yes)
+		(on_board yes)
+		(dnp no)
 		(fields_autoplaced yes)
 		(stroke
@@
 			(color 255 200 0 0.5020)
 		)
-		(property "Sheetname" "Section B - Title B"
+		(property "Sheetname" "Section B - Arduino Mega"
 			(at 190.5 113.2709 0)
 			(effects
@@
 		)
 		(instances
-			(project "KDT_Hierarchical_KiBot"
+			(project "VPDCU_EGSE"
 				(path "/f9e05184-c88b-4a88-ae9c-ab2bdb32be7c/c5103ceb-5325-4a84-a025-9638a412984e"
 					(page "5")
@@
 		(at 190.5 76.2)
 		(size 36.83 20.32)
+		(exclude_from_sim no)
+		(in_bom yes)
+		(on_board yes)
+		(dnp no)
 		(fields_autoplaced yes)
 		(stroke
@@
 			(color 128 255 128 0.5000)
 		)
-		(property "Sheetname" "Section A - Title A"
+		(property "Sheetname" "Section A - Connectors"
 			(at 190.5 75.1709 0)
 			(effects
@@
 		)
 		(instances
-			(project "KDT_Hierarchical_KiBot"
+			(project "VPDCU_EGSE"
 				(path "/f9e05184-c88b-4a88-ae9c-ab2bdb32be7c/c5103ceb-5325-4a84-a025-9638a412984e"
 					(page "4")
