File: Project Architecture.kicad_sch (KiCad schematic)
At the start: 0 parts

Commit message: PCB Checked version
Other:
- note added: "Page 6"
Changed lines of the file:
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@@
+		)
+	)
+	(text "Page 6"
+		(exclude_from_sim no)
+		(at 219.964 171.704 0)
+		(effects
+			(font
+				(size 2.54 2.54)
+				(thickness 0.508)
+				(bold yes)
+			)
+			(href "#6")
 		)
 	)
