File: Section A - Title A.kicad_sch (KiCad schematic)
At the start: 35 parts, among them J10 Conn_01x26, J11 L17HTHES4R1C, J12 DA15_Socket_MountingHoles, J13 FCR7350R, J14 FCR7350B, J15 DE09-SL-24, J25 KLDX-0202-A-LT, Q3 IRLZ44N, SW1 SW_Rotary_1x9_MP, T7 TestPoint, T8 TestPoint

Commit message: PCB Preliminary version
Parts:
- added T1, T10, T2, T3, T4, T5, T6, T9: TestPoint, TestPoint:TestPoint_Pad_1.0x1.0mm, symbol Connector:TestPoint
- J11: Manufacturer (none) -> Amphenol Communications Solutions; Manufacturer Part Number (none) -> L17HTHES4R1C; Manufacturer_Name Amphenol Communications Solutions -> (none); Manufacturer_Part_Number L17HTHES4R1C -> (none)
- T7, T8, VC1, VC2, VC3, VC4, VC5, VC6: footprint SamacSys_Parts:TestPoint_Pad_0.6x0.6mm -> TestPoint:TestPoint_Pad_1.0x1.0mm
Connections:
- net at J11.13: now also T9.1
- net at J11.15: now also T10.1
- net at J10.10 (Pin_10): now also T6.1
- net at J10.20 (Pin_20): now also T5.1
- net at J10.21 (Pin_21): now also T4.1
- net at J10.22 (Pin_22): now also T3.1
- net at J10.23 (Pin_23): now also T2.1
- net at J10.24 (Pin_24): now also T1.1
- no-connect marks 34 -> 26
Other:
- moved on the sheet: J10, J11, R33, R34, R35, R36, R38, R39, R40

Commit message: PCB Checked version
Parts:
- J10: Manufacturer Amphenol Positronic -> Amphenol ICC (Commercial Products); Manufacturer Part Number DD26S3S00S/AA -> L77HDA26SD1CH4F
- J11: footprint L17HTHES4R1C -> SamacSys_Parts:L17HTHES4R1C
- J12: footprint Connector_Dsub:DSUB-15-HD_Pins_Horizontal_P2.29x1.90mm_EdgePinOffset3.03mm_Housed_MountingHolesOffset4.94mm -> Library:AMPHENOL_10090926-P154XLF; Manufacturer (none) -> Amphenol ICC (FCI); Manufacturer Part Number (none) -> 10090926-P154XLF; Realtra Part Number (none) -> R-CON-1271-15PI
- J13: footprint FCR7350R -> SamacSys_Parts:FCR7350R; Manufacturer (none) -> CLIFF ELECTRONIC COMPONENTS; Manufacturer Part Number (none) -> FCR7350R; Manufacturer_Name CLIFF ELECTRONIC COMPONENTS -> (none); Manufacturer_Part_Number FCR7350R -> (none)
- J14: footprint FCR7350B -> SamacSys_Parts:FCR7350B; Manufacturer (none) -> CLIFF ELECTRONIC COMPONENTS; Manufacturer Part Number (none) -> FCR7350B; Manufacturer_Name CLIFF ELECTRONIC COMPONENTS -> (none); Manufacturer_Part_Number FCR7350B -> (none)
- J15: footprint DE09SL24 -> SamacSys_Parts:DE09SL24; Manufacturer (none) -> Adam Tech; Manufacturer Part Number (none) -> DE09-SL-24; Manufacturer_Name Adam Tech -> (none); Manufacturer_Part_Number DE09-SL-24 -> (none)
- J25: footprint KLDX0202ALT -> SamacSys_Parts:KLDX0202ALT; Manufacturer Name (none) -> Kycon; Manufacturer Part Number (none) -> KLDX-0202-A-LT; Manufacturer_Name Kycon -> (none); Manufacturer_Part_Number KLDX-0202-A-LT -> (none)
Other:
- title: Sheet Title A -> Power Entry and Connectors

Commit message: Schematic and PCB update
Parts:
- added H10, H11, H5, H6, H7, H8, H9: MountingHole_Pad_MP, MountingHole:MountingHole_3.2mm_M3_DIN965_Pad, symbol Mechanical:MountingHole_Pad_MP
- renumbered T8 to HTR_28V1, T7 to VDCU_28V1
Connections:
- net LD9_5V renamed HTR_28V
- net RX renamed RS232_RX_IN
- net TX renamed RS232_TX_OUT
- net VCAM_1 +28V renamed VCAM_1_28V
- net VCAM_2 +28V renamed VCAM_2_28V
- net VCAM_3 +28V renamed VCAM_3_28V
- net VCAM_4 +28V renamed VCAM_4_28V
- net VCAM_5 +28V renamed VCAM_5_28V
- net VCAM_6 +28V renamed VCAM_6_28V
- no-connect marks 26 -> 33
Other:
- note removed: "AN5346"
- note removed: "J. Pieper ADC investigation"
- note removed: "STM32G474 Datasheet p.81"
- moved on the sheet: C1, C2, H1, H2, H3, H4, J13, J14, J15, Q3, R41, R65
