File: Section C - Title C.kicad_sch (KiCad schematic)
At the start: 98 parts, among them J16 OSTOQ025450, J17 OSTOQ025450, J18 OSTOQ025450, J19 OSTOQ025450, J20 OSTOQ025450, J21 OSTOQ025450, J22 OSTOQ025450, J23 OSTOQ025450, J24 OSTOQ025450, J5 OSTOQ025450, K1 OJE-SH-105LMH,000, K10 OJE-SH-105LMH,000, K11 VOR1003M4T, K12 VOR1003M4T, K13 VOR1003M4T, K14 VOR1003M4T, K15 VOR1003M4T, K16 VOR1003M4T, K17 VOR1003M4T, K18 VOR1003M4T, K19 VOR1003M4T, K2 OJE-SH-105LMH,000, K20 VOR1003M4T, K3 OJE-SH-105LMH,000, K4 OJE-SH-105LMH,000, K5 OJE-SH-105LMH,000, K6 OJE-SH-105LMH,000, K7 OJE-SH-105LMH,000, K8 OJE-SH-105LMH,000, K9 OJE-SH-105LMH,000, Q10 IRLML2060, Q11 IRLML2060, Q12 IRLML2060, Q14 IRLML2060, Q15 IRLML2060, Q16 IRLML2060, Q17 IRLML2060, Q23 IRLML2060, Q24 IRLML2060, Q27 DMP6185SEQ-13, Q28 IRLML2060, Q29 IRLML2060, Q30 DMP6185SEQ-13, Q31 IRLML2060, Q32 DMP6185SEQ-13, Q33 IRLML2060, Q34 DMP6185SEQ-13, Q9 IRLML2060, T39 TestPoint, T40 TestPoint, T41 TestPoint, T42 TestPoint

Commit message: PCB Preliminary version
Parts:
- T39, T40, T41, T42: footprint SamacSys_Parts:TestPoint_Pad_0.6x0.6mm -> TestPoint:TestPoint_Pad_1.0x1.0mm
Other:
- moved on the sheet: C34, C35, C36, C37, J16, J17, J18, J19, J20, J21, J22, J23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

Commit message: PCB Checked version
Parts:
- J16, J17, J18, J19, J20, J21, J22, J23, J24, J5: footprint SHDR2W100P0X508_1X2_1216X860X1230P -> SamacSys_Parts:SHDR2W100P0X508_1X2_1216X860X1230P
- K1, K10, K2, K3, K4, K5, K6, K7, K8, K9: footprint OJESH105LMH000 -> SamacSys_Parts:OJESH105LMH000
- K11, K12, K13, K14, K15, K16, K17, K18, K19, K20: footprint VOR1003M4T -> SamacSys_Parts:VOR1003M4T
- Q27, Q30, Q32, Q34: footprint SOT230P700X180-4N -> SamacSys_Parts:SOT230P700X180-4N
Other:
- title: Sheet Title C -> LCL Selector

Commit message: Schematic and PCB update
Connections:
- net LD9_5V renamed HTR_28V
- net VCAM_1 +28V renamed VCAM_1_28V
- net VCAM_2 +28V renamed VCAM_2_28V
- net VCAM_3 +28V renamed VCAM_3_28V
- net VCAM_4 +28V renamed VCAM_4_28V
- net VCAM_5 +28V renamed VCAM_5_28V
- net VCAM_6 +28V renamed VCAM_6_28V
Other:
- note added: "HTR_28V"
- note added: "VCAM_1"
- note added: "VCAM_2"
- note added: "VCAM_3"
- note added: "VCAM_4"
- note added: "VCAM_5"
- note added: "VCAM_6"
- note added: "VDCU_28V"
- note added: "VTX_1"
- note added: "VTX_2"
- moved on the sheet: C34, C35, C36, C37, J16, J17, J18, J19, J20, J21, J22, J23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
